Commit message: Other Update

File: saps_ws/src/saps_bringup/urdf/saps_robot.xacro (robot description, xacro)
@@ -61,5 +61,5 @@
       <origin xyz="0 0 0" rpy="0 0 0"/>
       <geometry>
-        <box size="0.016 0.020 0.001"/>
+        <box size="0.028 0.028 0.001"/>
       </geometry>
       <material name="red">
@@ -70,5 +70,5 @@
       <origin xyz="0 0 0" rpy="0 0 0"/>
       <geometry>
-        <box size="0.016 0.020 0.001"/>
+        <box size="0.028 0.028 0.001"/>
       </geometry>
     </collision>
@@ -77,5 +77,5 @@
     <parent link="base_link"/>
     <child link="imu_link"/>
-    <origin xyz="0 0 ${base_height/2 - 0.002}" rpy="0 0 0"/>
+    <origin xyz="0 0 ${base_height/2 + 0.074}" rpy="0 0 0"/>
   </joint>
   <!-- ############ SENSORS ############ -->

Commit message: Etc UPdate

File: saps_ws/src/saps_bringup/urdf/saps_robot.xacro (robot description, xacro)
@@ -97,5 +97,5 @@
     <child link="camera_center_link"/>
     <!-- 로봇 앞쪽 중앙, 몸체 위 5cm에 위치. 실제 부착 위치에 맞게 자로 재서 수정하세요! -->
-    <origin xyz="${base_length/2 - 0.02} 0 ${base_height/2 + 0.02}" rpy="0 0 0"/>
+    <origin xyz="0.14 0 ${base_height/2 + 0.015}" rpy="0 0 0"/>
   </joint>
   <!-- 2. RealSense 드라이버가 기준점으로dd 사용하는 실제 '왼쪽 뎁스 렌즈'의 위치 -->
@@ -107,3 +107,4 @@
     <origin xyz="0 0.0475 0" rpy="0 0 0"/>
   </joint>
+  <!-- ####### Robot Arm ####### -->
 </robot>
